Commit message: change dae to stl

File: urdf/kr300r2500pro_macro.xacro (robot description, xacro)
@@ -14,6 +14,9 @@
         <origin xyz="0 0 0" rpy="0 0 0"/>
         <geometry>
-          <mesh filename="package://kuka_kr300_support/meshes/kr300r2500pro/visual/base_link.dae" />
-        </geometry>
+          <mesh filename="package://kuka_kr300_support/meshes/kr300r2500pro/visual/base_link.stl" />
+        </geometry>
+        <material name="">
+          <color rgba="1.0 1.0 1.0 1.0"/>
+        </material>
       </visual>
       <collision>
@@ -34,6 +37,9 @@
         <origin xyz="0 0 0" rpy="0 0 0"/>
         <geometry>
-          <mesh filename="package://kuka_kr300_support/meshes/kr300r2500pro/visual/link_1.dae" />
-        </geometry>
+          <mesh filename="package://kuka_kr300_support/meshes/kr300r2500pro/visual/link_1.stl" />
+        </geometry>
+        <material name="">
+          <color rgba="1.0 1.0 1.0 1.0"/>
+        </material>
       </visual>
       <collision>
@@ -54,6 +60,9 @@
         <origin xyz="0 0 0" rpy="0 0 0"/>
         <geometry>
-          <mesh filename="package://kuka_kr300_support/meshes/kr300r2500pro/visual/link_2.dae"/>
-        </geometry>
+          <mesh filename="package://kuka_kr300_support/meshes/kr300r2500pro/visual/link_2.stl"/>
+        </geometry>
+        <material name="">
+          <color rgba="1.0 1.0 1.0 1.0"/>
+        </material>
       </visual>
       <collision>
@@ -74,6 +83,9 @@
         <origin xyz="0 0 0" rpy="0 0 0"/>
         <geometry>
-          <mesh filename="package://kuka_kr300_support/meshes/kr300r2500pro/visual/link_3.dae" />
-        </geometry>
+          <mesh filename="package://kuka_kr300_support/meshes/kr300r2500pro/visual/link_3.stl" />
+        </geometry>
+        <material name="">
+          <color rgba="1.0 1.0 1.0 1.0"/>
+        </material>
       </visual>
       <collision>
@@ -94,6 +106,9 @@
         <origin xyz="0 0 0" rpy="0 0 0"/>
         <geometry>
-          <mesh filename="package://kuka_kr300_support/meshes/kr300r2500pro/visual/link_4.dae" />
-        </geometry>
+          <mesh filename="package://kuka_kr300_support/meshes/kr300r2500pro/visual/link_4.stl" />
+        </geometry>
+        <material name="">
+          <color rgba="1.0 1.0 1.0 1.0"/>
+        </material>
       </visual>
       <collision>
@@ -114,6 +129,9 @@
         <origin xyz="0 0 0" rpy="0 0 0"/>
         <geometry>
-          <mesh filename="package://kuka_kr300_support/meshes/kr300r2500pro/visual/link_5.dae" />
-        </geometry>
+          <mesh filename="package://kuka_kr300_support/meshes/kr300r2500pro/visual/link_5.stl" />
+        </geometry>
+        <material name="">
+          <color rgba="1.0 1.0 1.0 1.0"/>
+        </material>
       </visual>
       <collision>
@@ -134,6 +152,9 @@
         <origin xyz="0 0 0" rpy="0 0 0"/>
         <geometry>
-          <mesh filename="package://kuka_kr300_support/meshes/kr300r2500pro/visual/link_6.dae" />
-        </geometry>
+          <mesh filename="package://kuka_kr300_support/meshes/kr300r2500pro/visual/link_6.stl" />
+        </geometry>
+        <material name="">
+          <color rgba="1.0 1.0 1.0 1.0"/>
+        </material>
       </visual>
       <collision>

Commit message: comment  ROS base_link

File: urdf/kr300r2500pro_macro.xacro (robot description, xacro)
@@ -225,5 +225,5 @@
     </joint>
     <!-- END JOINTS -->
-    <!-- ROS base_link to KUKA $ROBROOT coordinate system transform -->
+    <!-- ROS base_link to KUKA $ROBROOT coordinate system transform >
     <link name="${prefix}base" />
     <joint name="${prefix}base_link-base" type="fixed">
@@ -231,5 +231,5 @@
       <parent link="${prefix}base_link"/>
       <child link="${prefix}base"/>
-    </joint>
+    </joint-->
   </xacro:macro>
 </robot>

Commit message: update mesh scale and use dae for visual

File: urdf/kr300r2500pro_macro.xacro (robot description, xacro)
@@ -14,14 +14,14 @@
         <origin xyz="0 0 0" rpy="0 0 0"/>
         <geometry>
-          <mesh filename="package://kuka_kr300_support/meshes/kr300r2500pro/visual/base_link.stl" />
-        </geometry>
-        <material name="">
-          <color rgba="1.0 1.0 1.0 1.0"/>
-        </material>
-      </visual>
-      <collision>
-        <origin xyz="0 0 0" rpy="0 0 0"/>
-        <geometry>
-          <mesh filename="package://kuka_kr300_support/meshes/kr300r2500pro/collision/base_link.stl" />
+          <mesh scale="0.001 0.001 0.001" filename="package://kuka_kr300_support/meshes/kr300r2500pro/visual/base_link.dae" />
+        </geometry>
+        <material name="">
+          <color rgba="1.0 1.0 1.0 1.0"/>
+        </material>
+      </visual>
+      <collision>
+        <origin xyz="0 0 0" rpy="0 0 0"/>
+        <geometry>
+          <mesh scale="0.001 0.001 0.001" filename="package://kuka_kr300_support/meshes/kr300r2500pro/collision/base_link.stl" />
         </geometry>
       </collision>
@@ -37,14 +37,14 @@
         <origin xyz="0 0 0" rpy="0 0 0"/>
         <geometry>
-          <mesh filename="package://kuka_kr300_support/meshes/kr300r2500pro/visual/link_1.stl" />
-        </geometry>
-        <material name="">
-          <color rgba="1.0 1.0 1.0 1.0"/>
-        </material>
-      </visual>
-      <collision>
-        <origin xyz="0 0 0" rpy="0 0 0"/>
-        <geometry>
-          <mesh filename="package://kuka_kr300_support/meshes/kr300r2500pro/collision/link_1.stl" />
+          <mesh scale="0.001 0.001 0.001" filename="package://kuka_kr300_support/meshes/kr300r2500pro/visual/link_1.dae" />
+        </geometry>
+        <material name="">
+          <color rgba="1.0 1.0 1.0 1.0"/>
+        </material>
+      </visual>
+      <collision>
+        <origin xyz="0 0 0" rpy="0 0 0"/>
+        <geometry>
+          <mesh scale="0.001 0.001 0.001" filename="package://kuka_kr300_support/meshes/kr300r2500pro/collision/link_1.stl" />
         </geometry>
       </collision>
@@ -60,14 +60,14 @@
         <origin xyz="0 0 0" rpy="0 0 0"/>
         <geometry>
-          <mesh filename="package://kuka_kr300_support/meshes/kr300r2500pro/visual/link_2.stl"/>
-        </geometry>
-        <material name="">
-          <color rgba="1.0 1.0 1.0 1.0"/>
-        </material>
-      </visual>
-      <collision>
-        <origin xyz="0 0 0" rpy="0 0 0"/>
-        <geometry>
-          <mesh filename="package://kuka_kr300_support/meshes/kr300r2500pro/collision/link_2.stl" />
+          <mesh scale="0.001 0.001 0.001" filename="package://kuka_kr300_support/meshes/kr300r2500pro/visual/link_2.dae"/>
+        </geometry>
+        <material name="">
+          <color rgba="1.0 1.0 1.0 1.0"/>
+        </material>
+      </visual>
+      <collision>
+        <origin xyz="0 0 0" rpy="0 0 0"/>
+        <geometry>
+          <mesh scale="0.001 0.001 0.001" filename="package://kuka_kr300_support/meshes/kr300r2500pro/collision/link_2.stl" />
         </geometry>
       </collision>
@@ -83,14 +83,14 @@
         <origin xyz="0 0 0" rpy="0 0 0"/>
         <geometry>
-          <mesh filename="package://kuka_kr300_support/meshes/kr300r2500pro/visual/link_3.stl" />
-        </geometry>
-        <material name="">
-          <color rgba="1.0 1.0 1.0 1.0"/>
-        </material>
-      </visual>
-      <collision>
-        <origin xyz="0 0 0" rpy="0 0 0"/>
-        <geometry>
-          <mesh filename="package://kuka_kr300_support/meshes/kr300r2500pro/collision/link_3.stl" />
+          <mesh scale="0.001 0.001 0.001" filename="package://kuka_kr300_support/meshes/kr300r2500pro/visual/link_3.dae" />
+        </geometry>
+        <material name="">
+          <color rgba="1.0 1.0 1.0 1.0"/>
+        </material>
+      </visual>
+      <collision>
+        <origin xyz="0 0 0" rpy="0 0 0"/>
+        <geometry>
+          <mesh scale="0.001 0.001 0.001" filename="package://kuka_kr300_support/meshes/kr300r2500pro/collision/link_3.stl" />
         </geometry>
       </collision>
@@ -106,14 +106,14 @@
         <origin xyz="0 0 0" rpy="0 0 0"/>
         <geometry>
-          <mesh filename="package://kuka_kr300_support/meshes/kr300r2500pro/visual/link_4.stl" />
-        </geometry>
-        <material name="">
-          <color rgba="1.0 1.0 1.0 1.0"/>
-        </material>
-      </visual>
-      <collision>
-        <origin xyz="0 0 0" rpy="0 0 0"/>
-        <geometry>
-          <mesh filename="package://kuka_kr300_support/meshes/kr300r2500pro/collision/link_4.stl" />
+          <mesh scale="0.001 0.001 0.001" filename="package://kuka_kr300_support/meshes/kr300r2500pro/visual/link_4.dae" />
+        </geometry>
+        <material name="">
+          <color rgba="1.0 1.0 1.0 1.0"/>
+        </material>
+      </visual>
+      <collision>
+        <origin xyz="0 0 0" rpy="0 0 0"/>
+        <geometry>
+          <mesh scale="0.001 0.001 0.001" filename="package://kuka_kr300_support/meshes/kr300r2500pro/collision/link_4.stl" />
         </geometry>
       </collision>
@@ -129,14 +129,14 @@
         <origin xyz="0 0 0" rpy="0 0 0"/>
         <geometry>
-          <mesh filename="package://kuka_kr300_support/meshes/kr300r2500pro/visual/link_5.stl" />
-        </geometry>
-        <material name="">
-          <color rgba="1.0 1.0 1.0 1.0"/>
-        </material>
-      </visual>
-      <collision>
-        <origin xyz="0 0 0" rpy="0 0 0"/>
-        <geometry>
-          <mesh filename="package://kuka_kr300_support/meshes/kr300r2500pro/collision/link_5.stl" />
+          <mesh scale="0.001 0.001 0.001" filename="package://kuka_kr300_support/meshes/kr300r2500pro/visual/link_5.dae" />
+        </geometry>
+        <material name="">
+          <color rgba="1.0 1.0 1.0 1.0"/>
+        </material>
+      </visual>
+      <collision>
+        <origin xyz="0 0 0" rpy="0 0 0"/>
+        <geometry>
+          <mesh scale="0.001 0.001 0.001" filename="package://kuka_kr300_support/meshes/kr300r2500pro/collision/link_5.stl" />
         </geometry>
       </collision>
@@ -152,14 +152,14 @@
         <origin xyz="0 0 0" rpy="0 0 0"/>
         <geometry>
-          <mesh filename="package://kuka_kr300_support/meshes/kr300r2500pro/visual/link_6.stl" />
-        </geometry>
-        <material name="">
-          <color rgba="1.0 1.0 1.0 1.0"/>
-        </material>
-      </visual>
-      <collision>
-        <origin xyz="0 0 0" rpy="0 0 0"/>
-        <geometry>
-          <mesh filename="package://kuka_kr300_support/meshes/kr300r2500pro/collision/link_6.stl" />
+          <mesh scale="0.001 0.001 0.001" filename="package://kuka_kr300_support/meshes/kr300r2500pro/visual/link_6.dae" />
+        </geometry>
+        <material name="">
+          <color rgba="1.0 1.0 1.0 1.0"/>
+        </material>
+      </visual>
+      <collision>
+        <origin xyz="0 0 0" rpy="0 0 0"/>
+        <geometry>
+          <mesh scale="0.001 0.001 0.001" filename="package://kuka_kr300_support/meshes/kr300r2500pro/collision/link_6.stl" />
         </geometry>
       </collision>

Commit message: set visualization mesh file format to STL

File: urdf/kr300r2500pro_macro.xacro (robot description, xacro)
@@ -14,5 +14,5 @@
         <origin xyz="0 0 0" rpy="0 0 0"/>
         <geometry>
-          <mesh scale="0.001 0.001 0.001" filename="package://kuka_kr300_support/meshes/kr300r2500pro/visual/base_link.dae" />
+          <mesh filename="package://kuka_kr300_support/meshes/kr300r2500pro/visual/base_link.stl" />
         </geometry>
         <material name="">
@@ -37,5 +37,5 @@
         <origin xyz="0 0 0" rpy="0 0 0"/>
         <geometry>
-          <mesh scale="0.001 0.001 0.001" filename="package://kuka_kr300_support/meshes/kr300r2500pro/visual/link_1.dae" />
+          <mesh filename="package://kuka_kr300_support/meshes/kr300r2500pro/visual/link_1.stl" />
         </geometry>
         <material name="">
@@ -60,5 +60,5 @@
         <origin xyz="0 0 0" rpy="0 0 0"/>
         <geometry>
-          <mesh scale="0.001 0.001 0.001" filename="package://kuka_kr300_support/meshes/kr300r2500pro/visual/link_2.dae"/>
+          <mesh filename="package://kuka_kr300_support/meshes/kr300r2500pro/visual/link_2.stl"/>
         </geometry>
         <material name="">
@@ -83,5 +83,5 @@
         <origin xyz="0 0 0" rpy="0 0 0"/>
         <geometry>
-          <mesh scale="0.001 0.001 0.001" filename="package://kuka_kr300_support/meshes/kr300r2500pro/visual/link_3.dae" />
+          <mesh filename="package://kuka_kr300_support/meshes/kr300r2500pro/visual/link_3.stl" />
         </geometry>
         <material name="">
@@ -106,5 +106,5 @@
         <origin xyz="0 0 0" rpy="0 0 0"/>
         <geometry>
-          <mesh scale="0.001 0.001 0.001" filename="package://kuka_kr300_support/meshes/kr300r2500pro/visual/link_4.dae" />
+          <mesh filename="package://kuka_kr300_support/meshes/kr300r2500pro/visual/link_4.stl" />
         </geometry>
         <material name="">
@@ -129,5 +129,5 @@
         <origin xyz="0 0 0" rpy="0 0 0"/>
         <geometry>
-          <mesh scale="0.001 0.001 0.001" filename="package://kuka_kr300_support/meshes/kr300r2500pro/visual/link_5.dae" />
+          <mesh filename="package://kuka_kr300_support/meshes/kr300r2500pro/visual/link_5.stl" />
         </geometry>
         <material name="">
@@ -152,5 +152,5 @@
         <origin xyz="0 0 0" rpy="0 0 0"/>
         <geometry>
-          <mesh scale="0.001 0.001 0.001" filename="package://kuka_kr300_support/meshes/kr300r2500pro/visual/link_6.dae" />
+          <mesh filename="package://kuka_kr300_support/meshes/kr300r2500pro/visual/link_6.stl" />
         </geometry>
         <material name="">
