Commit message: remove ROS base link

File: urdf/kr300r2500pro.urdf (robot description, URDF)
Before this commit: robot kuka_kr300r2500pro, 0 links, 0 joints
Links:
- added link base_link, mass 2; collision mesh filename=package://kuka_kr300_support/meshes/kr300r2500pro/collision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; visual mesh filename=package://kuka_kr300_support/meshes/kr300r2500pro/visual/ba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
- added link link_1, mass 2; collision mesh filename=package://kuka_kr300_support/meshes/kr300r2500pro/collision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; visual mesh filename=package://kuka_kr300_support/meshes/kr300r2500pro/visual/li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
- added link link_2, mass 2; collision mesh filename=package://kuka_kr300_support/meshes/kr300r2500pro/collision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; visual mesh filename=package://kuka_kr300_support/meshes/kr300r2500pro/visual/li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
- added link link_3, mass 2; collision mesh filename=package://kuka_kr300_support/meshes/kr300r2500pro/collision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; visual mesh filename=package://kuka_kr300_support/meshes/kr300r2500pro/visual/li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
- added link link_4, mass 2; collision mesh filename=package://kuka_kr300_support/meshes/kr300r2500pro/collision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; visual mesh filename=package://kuka_kr300_support/meshes/kr300r2500pro/visual/li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
- added link link_5, mass 2; collision mesh filename=package://kuka_kr300_support/meshes/kr300r2500pro/collision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; visual mesh filename=package://kuka_kr300_support/meshes/kr300r2500pro/visual/li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
- added link link_6, mass 2; collision mesh filename=package://kuka_kr300_support/meshes/kr300r2500pro/collision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; visual mesh filename=package://kuka_kr300_support/meshes/kr300r2500pro/visual/li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
- added link tool0
Joints:
- added joint joint_a1: type revolute, parent base_link, child link_1, origin xyz=0 0 0.675 rpy=0 0 0, axis 0 0 -1, limit lower=-3.2288591161895095 upper=3.2288591161895095 effort=0 velocity=2.722713633111154
- added joint joint_a2: type revolute, parent link_1, child link_2, origin xyz=0.35 0 0 rpy=0 0 0, axis 0 1 0, limit lower=-2.705260340591211 upper=0.6108652381980153 effort=0 velocity=2.722713633111154
- added joint joint_a3: type revolute, parent link_2, child link_3, origin xyz=1.150 0 0 rpy=0 0 0, axis 0 1 0, limit lower=-2.2689280275926285 upper=2.6878070480712677 effort=0 velocity=2.722713633111154
- added joint joint_a4: type revolute, parent link_3, child link_4, origin xyz=1.0 0 -0.041 rpy=0 0 0, axis -1 0 0, limit lower=-6.1086523819801535 upper=6.1086523819801535 effort=0 velocity=5.759586531581287
- added joint joint_a5: type revolute, parent link_4, child link_5, origin xyz=0 0 0 rpy=0 0 0, axis 0 1 0, limit lower=-2.2689280275926285 upper=2.2689280275926285 effort=0 velocity=5.759586531581287
- added joint joint_a6: type revolute, parent link_5, child link_6, origin xyz=0 0 0 rpy=0 0 0, axis -1 0 0, limit lower=-6.1086523819801535 upper=6.1086523819801535 effort=0 velocity=10.733774899765127
- added joint joint_a6-tool0: type fixed, parent link_6, child tool0, origin xyz=0.240 0 0 rpy=0 1.5707963267948966 0

Commit message: updated mesh

File: urdf/kr300r2500pro.urdf (robot description, URDF)
Before this commit: robot kuka_kr300r2500pro, 0 links, 0 joints
Links:
- added link base
- added link base_link, mass 2; collision mesh filename=package://kuka_kr300_support/meshes/kr300r2500pro/collision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 scale=0.001 0.001 0.001; visual mesh filename=package://kuka_kr300_support/meshes/kr300r2500pro/visual/ba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
- added link link_1, mass 2; collision mesh filename=package://kuka_kr300_support/meshes/kr300r2500pro/collision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 scale=0.001 0.001 0.001; visual mesh filename=package://kuka_kr300_support/meshes/kr300r2500pro/visual/li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
- added link link_2, mass 2; collision mesh filename=package://kuka_kr300_support/meshes/kr300r2500pro/collision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 scale=0.001 0.001 0.001; visual mesh filename=package://kuka_kr300_support/meshes/kr300r2500pro/visual/li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
- added link link_3, mass 2; collision mesh filename=package://kuka_kr300_support/meshes/kr300r2500pro/collision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 scale=0.001 0.001 0.001; visual mesh filename=package://kuka_kr300_support/meshes/kr300r2500pro/visual/li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
- added link link_4, mass 2; collision mesh filename=package://kuka_kr300_support/meshes/kr300r2500pro/collision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 scale=0.001 0.001 0.001; visual mesh filename=package://kuka_kr300_support/meshes/kr300r2500pro/visual/li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
- added link link_5, mass 2; collision mesh filename=package://kuka_kr300_support/meshes/kr300r2500pro/collision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 scale=0.001 0.001 0.001; visual mesh filename=package://kuka_kr300_support/meshes/kr300r2500pro/visual/li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
- added link link_6, mass 2; collision mesh filename=package://kuka_kr300_support/meshes/kr300r2500pro/collision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 scale=0.001 0.001 0.001; visual mesh filename=package://kuka_kr300_support/meshes/kr300r2500pro/visual/li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
- added link tool0
Joints:
- added joint base_link-base: type fixed, parent base_link, child base, origin xyz=0 0 0 rpy=0 0 0
- added joint joint_a1: type revolute, parent base_link, child link_1, origin xyz=0 0 0.675 rpy=0 0 0, axis 0 0 -1, limit lower=-3.2288591161895095 upper=3.2288591161895095 effort=0 velocity=2.722713633111154
- added joint joint_a2: type revolute, parent link_1, child link_2, origin xyz=0.35 0 0 rpy=0 0 0, axis 0 1 0, limit lower=-2.705260340591211 upper=0.6108652381980153 effort=0 velocity=2.722713633111154
- added joint joint_a3: type revolute, parent link_2, child link_3, origin xyz=1.150 0 0 rpy=0 0 0, axis 0 1 0, limit lower=-2.2689280275926285 upper=2.6878070480712677 effort=0 velocity=2.722713633111154
- added joint joint_a4: type revolute, parent link_3, child link_4, origin xyz=1.0 0 -0.041 rpy=0 0 0, axis -1 0 0, limit lower=-6.1086523819801535 upper=6.1086523819801535 effort=0 velocity=5.759586531581287
- added joint joint_a5: type revolute, parent link_4, child link_5, origin xyz=0 0 0 rpy=0 0 0, axis 0 1 0, limit lower=-2.2689280275926285 upper=2.2689280275926285 effort=0 velocity=5.759586531581287
- added joint joint_a6: type revolute, parent link_5, child link_6, origin xyz=0 0 0 rpy=0 0 0, axis -1 0 0, limit lower=-6.1086523819801535 upper=6.1086523819801535 effort=0 velocity=10.733774899765127
- added joint joint_a6-tool0: type fixed, parent link_6, child tool0, origin xyz=0.240 0 0 rpy=0 1.5707963267948966 0
