Commit message: rename kr300r2500pro to kr300r2500ultra

File: urdf/kr300r2500ultra.urdf (robot description, URDF)
Before this commit: robot kuka_kr300r2500pro, 9 links, 8 joints
Links:
- link base_link: geometry collision mesh filename=package://kuka_kr300_support/meshes/kr300r2500ultra/collisi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 scale=0.001 0.001 0.001; visual mesh filename=package://kuka_kr300_support/meshes/kr300r2500ultra/visual/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
- link link_1: geometry collision mesh filename=package://kuka_kr300_support/meshes/kr300r2500ultra/collisi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 scale=0.001 0.001 0.001; visual mesh filename=package://kuka_kr300_support/meshes/kr300r2500ultra/visual/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
- link link_2: geometry collision mesh filename=package://kuka_kr300_support/meshes/kr300r2500ultra/collisi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 scale=0.001 0.001 0.001; visual mesh filename=package://kuka_kr300_support/meshes/kr300r2500ultra/visual/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
- link link_3: geometry collision mesh filename=package://kuka_kr300_support/meshes/kr300r2500ultra/collisi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 scale=0.001 0.001 0.001; visual mesh filename=package://kuka_kr300_support/meshes/kr300r2500ultra/visual/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
- link link_4: geometry collision mesh filename=package://kuka_kr300_support/meshes/kr300r2500ultra/collisi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 scale=0.001 0.001 0.001; visual mesh filename=package://kuka_kr300_support/meshes/kr300r2500ultra/visual/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
- link link_5: geometry collision mesh filename=package://kuka_kr300_support/meshes/kr300r2500ultra/collisi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 scale=0.001 0.001 0.001; visual mesh filename=package://kuka_kr300_support/meshes/kr300r2500ultra/visual/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
- link link_6: geometry collision mesh filename=package://kuka_kr300_support/meshes/kr300r2500ultra/collisi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 scale=0.001 0.001 0.001; visual mesh filename=package://kuka_kr300_support/meshes/kr300r2500ultra/visual/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

File: urdf/kr300r2500ultra_macro.xacro (robot description, xacro)
@@ -2,5 +2,5 @@
 <robot xmlns:xacro="http://wiki.ros.org/xacro">
   <xacro:property name="DEG2RAD" value="0.017453292519943295"/>
-  <xacro:macro name="kuka_kr300r2500pro" params="prefix">
+  <xacro:macro name="kuka_kr300r2500ultra" params="prefix">
     <!-- LINKS -->
     <!-- base link -->
@@ -14,14 +14,14 @@
         <origin xyz="0 0 0" rpy="0 0 0"/>
         <geometry>
-          <mesh filename="package://kuka_kr300_support/meshes/kr300r2500pro/visual/base_link.stl" />
-        </geometry>
-        <material name="">
-          <color rgba="1.0 1.0 1.0 1.0"/>
-        </material>
-      </visual>
-      <collision>
-        <origin xyz="0 0 0" rpy="0 0 0"/>
-        <geometry>
-          <mesh scale="0.001 0.001 0.001" filename="package://kuka_kr300_support/meshes/kr300r2500pro/collision/base_link.stl" />
+          <mesh filename="package://kuka_kr300_support/meshes/kr300r2500ultra/visual/base_link.stl" />
+        </geometry>
+        <material name="">
+          <color rgba="1.0 1.0 1.0 1.0"/>
+        </material>
+      </visual>
+      <collision>
+        <origin xyz="0 0 0" rpy="0 0 0"/>
+        <geometry>
+          <mesh scale="0.001 0.001 0.001" filename="package://kuka_kr300_support/meshes/kr300r2500ultra/collision/base_link.stl" />
         </geometry>
       </collision>
@@ -37,14 +37,14 @@
         <origin xyz="0 0 0" rpy="0 0 0"/>
         <geometry>
-          <mesh filename="package://kuka_kr300_support/meshes/kr300r2500pro/visual/link_1.stl" />
-        </geometry>
-        <material name="">
-          <color rgba="1.0 1.0 1.0 1.0"/>
-        </material>
-      </visual>
-      <collision>
-        <origin xyz="0 0 0" rpy="0 0 0"/>
-        <geometry>
-          <mesh scale="0.001 0.001 0.001" filename="package://kuka_kr300_support/meshes/kr300r2500pro/collision/link_1.stl" />
+          <mesh filename="package://kuka_kr300_support/meshes/kr300r2500ultra/visual/link_1.stl" />
+        </geometry>
+        <material name="">
+          <color rgba="1.0 1.0 1.0 1.0"/>
+        </material>
+      </visual>
+      <collision>
+        <origin xyz="0 0 0" rpy="0 0 0"/>
+        <geometry>
+          <mesh scale="0.001 0.001 0.001" filename="package://kuka_kr300_support/meshes/kr300r2500ultra/collision/link_1.stl" />
         </geometry>
       </collision>
@@ -60,14 +60,14 @@
         <origin xyz="0 0 0" rpy="0 0 0"/>
         <geometry>
-          <mesh filename="package://kuka_kr300_support/meshes/kr300r2500pro/visual/link_2.stl"/>
-        </geometry>
-        <material name="">
-          <color rgba="1.0 1.0 1.0 1.0"/>
-        </material>
-      </visual>
-      <collision>
-        <origin xyz="0 0 0" rpy="0 0 0"/>
-        <geometry>
-          <mesh scale="0.001 0.001 0.001" filename="package://kuka_kr300_support/meshes/kr300r2500pro/collision/link_2.stl" />
+          <mesh filename="package://kuka_kr300_support/meshes/kr300r2500ultra/visual/link_2.stl"/>
+        </geometry>
+        <material name="">
+          <color rgba="1.0 1.0 1.0 1.0"/>
+        </material>
+      </visual>
+      <collision>
+        <origin xyz="0 0 0" rpy="0 0 0"/>
+        <geometry>
+          <mesh scale="0.001 0.001 0.001" filename="package://kuka_kr300_support/meshes/kr300r2500ultra/collision/link_2.stl" />
         </geometry>
       </collision>
@@ -83,14 +83,14 @@
         <origin xyz="0 0 0" rpy="0 0 0"/>
         <geometry>
-          <mesh filename="package://kuka_kr300_support/meshes/kr300r2500pro/visual/link_3.stl" />
-        </geometry>
-        <material name="">
-          <color rgba="1.0 1.0 1.0 1.0"/>
-        </material>
-      </visual>
-      <collision>
-        <origin xyz="0 0 0" rpy="0 0 0"/>
-        <geometry>
-          <mesh scale="0.001 0.001 0.001" filename="package://kuka_kr300_support/meshes/kr300r2500pro/collision/link_3.stl" />
+          <mesh filename="package://kuka_kr300_support/meshes/kr300r2500ultra/visual/link_3.stl" />
+        </geometry>
+        <material name="">
+          <color rgba="1.0 1.0 1.0 1.0"/>
+        </material>
+      </visual>
+      <collision>
+        <origin xyz="0 0 0" rpy="0 0 0"/>
+        <geometry>
+          <mesh scale="0.001 0.001 0.001" filename="package://kuka_kr300_support/meshes/kr300r2500ultra/collision/link_3.stl" />
         </geometry>
       </collision>
@@ -106,14 +106,14 @@
         <origin xyz="0 0 0" rpy="0 0 0"/>
         <geometry>
-          <mesh filename="package://kuka_kr300_support/meshes/kr300r2500pro/visual/link_4.stl" />
-        </geometry>
-        <material name="">
-          <color rgba="1.0 1.0 1.0 1.0"/>
-        </material>
-      </visual>
-      <collision>
-        <origin xyz="0 0 0" rpy="0 0 0"/>
-        <geometry>
-          <mesh scale="0.001 0.001 0.001" filename="package://kuka_kr300_support/meshes/kr300r2500pro/collision/link_4.stl" />
+          <mesh filename="package://kuka_kr300_support/meshes/kr300r2500ultra/visual/link_4.stl" />
+        </geometry>
+        <material name="">
+          <color rgba="1.0 1.0 1.0 1.0"/>
+        </material>
+      </visual>
+      <collision>
+        <origin xyz="0 0 0" rpy="0 0 0"/>
+        <geometry>
+          <mesh scale="0.001 0.001 0.001" filename="package://kuka_kr300_support/meshes/kr300r2500ultra/collision/link_4.stl" />
         </geometry>
       </collision>
@@ -129,14 +129,14 @@
         <origin xyz="0 0 0" rpy="0 0 0"/>
         <geometry>
-          <mesh filename="package://kuka_kr300_support/meshes/kr300r2500pro/visual/link_5.stl" />
-        </geometry>
-        <material name="">
-          <color rgba="1.0 1.0 1.0 1.0"/>
-        </material>
-      </visual>
-      <collision>
-        <origin xyz="0 0 0" rpy="0 0 0"/>
-        <geometry>
-          <mesh scale="0.001 0.001 0.001" filename="package://kuka_kr300_support/meshes/kr300r2500pro/collision/link_5.stl" />
+          <mesh filename="package://kuka_kr300_support/meshes/kr300r2500ultra/visual/link_5.stl" />
+        </geometry>
+        <material name="">
+          <color rgba="1.0 1.0 1.0 1.0"/>
+        </material>
+      </visual>
+      <collision>
+        <origin xyz="0 0 0" rpy="0 0 0"/>
+        <geometry>
+          <mesh scale="0.001 0.001 0.001" filename="package://kuka_kr300_support/meshes/kr300r2500ultra/collision/link_5.stl" />
         </geometry>
       </collision>
@@ -152,14 +152,14 @@
         <origin xyz="0 0 0" rpy="0 0 0"/>
         <geometry>
-          <mesh filename="package://kuka_kr300_support/meshes/kr300r2500pro/visual/link_6.stl" />
-        </geometry>
-        <material name="">
-          <color rgba="1.0 1.0 1.0 1.0"/>
-        </material>
-      </visual>
-      <collision>
-        <origin xyz="0 0 0" rpy="0 0 0"/>
-        <geometry>
-          <mesh scale="0.001 0.001 0.001" filename="package://kuka_kr300_support/meshes/kr300r2500pro/collision/link_6.stl" />
+          <mesh filename="package://kuka_kr300_support/meshes/kr300r2500ultra/visual/link_6.stl" />
+        </geometry>
+        <material name="">
+          <color rgba="1.0 1.0 1.0 1.0"/>
+        </material>
+      </visual>
+      <collision>
+        <origin xyz="0 0 0" rpy="0 0 0"/>
+        <geometry>
+          <mesh scale="0.001 0.001 0.001" filename="package://kuka_kr300_support/meshes/kr300r2500ultra/collision/link_6.stl" />
         </geometry>
       </collision>
